Commit message: add map server launch

File: Section4_Sensors_for_Localization_and_Mapping/bumperbot_ws/src/bumperbot_description/urdf/bumperbot_gazebo.xacro (robot description, xacro)
@@ -18,4 +18,5 @@
   <!-- Wheels -->
   <gazebo reference="wheel_left_link">
+    <material>Gazebo/Blue</material>
     <mu1>1000000000000000.0</mu1>
     <mu2>1000000000000000.0</mu2>
@@ -27,4 +28,5 @@
   </gazebo>
   <gazebo reference="wheel_right_link">
+    <material>Gazebo/Blue</material>
     <mu1>1000000000000000.0</mu1>
     <mu2>1000000000000000.0</mu2>
@@ -37,4 +39,5 @@
   <!-- Caster Wheels -->
   <gazebo reference="caster_rear_link">
+    <material>Gazebo/FlatBlack</material>
     <mu1>0.1</mu1>
     <mu2>0.1</mu2>
@@ -45,4 +48,5 @@
   </gazebo>
   <gazebo reference="caster_front_link">
+    <material>Gazebo/FlatBlack</material>
     <mu1>0.1</mu1>
     <mu2>0.1</mu2>
@@ -51,4 +55,10 @@
     <minDepth>0.001</minDepth>
     <maxVel>1.0</maxVel>
+  </gazebo>
+  <gazebo reference="base_link">
+    <material>Gazebo/FlatBlack</material>
+  </gazebo>
+  <gazebo reference="laser_link">
+    <material>Gazebo/FlatBlack</material>
   </gazebo>
   <!-- ROS 2 Control -->
