Commit message: update laser link based on real robot

File: Section10_SLAM/bumperbot_ws/src/bumperbot_description/urdf/bumperbot.urdf.xacro (robot description, xacro)
@@ -192,5 +192,5 @@
   </link>
   <joint name="laser_joint" type="fixed">
-    <origin xyz="-0.0050526 -0.0023221 0.1208" rpy="0 0 0" />
+    <origin xyz="-0.0050526 -0.0023221 0.1208" rpy="0 0 3.14" />
     <parent link="base_link" />
     <child link="laser_link" />
