Commit message: aupdate section9 with new Gazebo

File: Section9_Localization_with_known_Map/bumperbot_ws/src/bumperbot_description/urdf/bumperbot.urdf.xacro (robot description, xacro)
@@ -1,4 +1,6 @@
 <?xml version="1.0"?>
 <robot name="bumperbot" xmlns:xacro="http://ros.org/wiki/xacro">
+  <!-- Start GZ or Ignition depending on ROS 2 Version -->
+  <xacro:arg name="is_ignition" default="true"/>
   <!-- Load Simulated or Real Hardware Interfaces -->
   <xacro:arg name="is_sim" default="true"/>
@@ -11,5 +13,5 @@
     <inertial>
       <origin xyz="0 0 0.04" rpy="0.0 0.25 0.3" />
-      <mass value="1.0"/>
+      <mass value="8.2573504e-01"/>
       <inertia ixx="2.2124416e-02" ixy="-1.2294101e-04" ixz="3.4938785e-04"
                iyy="2.1193702e-02" iyz="-5.0120904e-05"
@@ -37,5 +39,5 @@
     <inertial>
       <origin xyz="0 -0.014 0" rpy="0 0 0" />
-      <mass value="1.0" />
+      <mass value="0.0530086090966721" />
       <inertia ixx="1.88176298336665E-05" ixy="-4.8444933029987E-10" ixz="1.88163708851143E-08"
                iyy="3.11510738647764E-05" iyz="-6.93560663069607E-11"
@@ -65,5 +67,5 @@
     <inertial>
       <origin xyz="0 0.014 0" rpy="0 0 0" />
-      <mass value="1.0" />
+      <mass value="0.0530086043217644" />
       <inertia ixx="1.8792911368909E-05"  ixy="3.31256392204584E-10" ixz="-1.14082001662767E-08"
                iyy="3.11510738759073E-05" iyz="-3.60499245082192E-10"
@@ -156,4 +158,7 @@
         <mesh filename="package://bumperbot_description/meshes/imu_link.STL" />
       </geometry>
+      <material name="">
+        <color rgba="0.792156862745098 0.819607843137255 0.933333333333333 1" />
+      </material>
     </visual>
     <collision>

File: Section9_Localization_with_known_Map/bumperbot_ws/src/bumperbot_description/urdf/bumperbot_gazebo.xacro (robot description, xacro)
@@ -1,22 +1,6 @@
 <?xml version="1.0"?>
 <robot name="bumperbot" xmlns:xacro="http://ros.org/wiki/xacro">
-  <!-- Move this one to ros2 control -->
-  <transmission name="wheel_right_transmission">
-    <plugin>transmission_interface/SimpleTransmission</plugin>
-    <actuator name="wheel_right_motor" role="actuator_right"/>
-    <joint name="wheel_right_joint"    role="joint_right">
-      <mechanical_reduction>1.0</mechanical_reduction>
-    </joint>
-  </transmission>
-  <transmission name="wheel_left_transmission">
-    <plugin>transmission_interface/SimpleTransmission</plugin>
-    <actuator name="wheel_left_motor" role="actuator_left"/>
-    <joint name="wheel_left_joint"    role="joint_left">
-      <mechanical_reduction>1.0</mechanical_reduction>
-    </joint>
-  </transmission>
   <!-- Wheels -->
   <gazebo reference="wheel_left_link">
-    <material>Gazebo/Blue</material>
     <mu1>1000000000000000.0</mu1>
     <mu2>1000000000000000.0</mu2>
@@ -28,5 +12,4 @@
   </gazebo>
   <gazebo reference="wheel_right_link">
-    <material>Gazebo/Blue</material>
     <mu1>1000000000000000.0</mu1>
     <mu2>1000000000000000.0</mu2>
@@ -39,5 +22,4 @@
   <!-- Caster Wheels -->
   <gazebo reference="caster_rear_link">
-    <material>Gazebo/FlatBlack</material>
     <mu1>0.1</mu1>
     <mu2>0.1</mu2>
@@ -48,5 +30,4 @@
   </gazebo>
   <gazebo reference="caster_front_link">
-    <material>Gazebo/FlatBlack</material>
     <mu1>0.1</mu1>
     <mu2>0.1</mu2>
@@ -56,17 +37,28 @@
     <maxVel>1.0</maxVel>
   </gazebo>
-  <gazebo reference="base_link">
-    <material>Gazebo/FlatBlack</material>
-  </gazebo>
-  <gazebo reference="laser_link">
-    <material>Gazebo/FlatBlack</material>
-  </gazebo>
   <!-- ROS 2 Control -->
   <gazebo>
-    <plugin filename="libgazebo_ros2_control.so" name="gazebo_ros2_control">
-      <robot_param>robot_description</robot_param>
-      <robot_param_node>robot_state_publisher</robot_param_node>
-      <parameters>$(find bumperbot_controller)/config/bumperbot_controllers.yaml</parameters>
-    </plugin>
+    <!-- ROS 2 Humble -->
+    <xacro:if value="$(arg is_ignition)">
+      <plugin filename="ign_ros2_control-system" name="ign_ros2_control::IgnitionROS2ControlPlugin">
+        <parameters>$(find bumperbot_controller)/config/bumperbot_controllers.yaml</parameters>
+      </plugin>
+      <plugin filename="ignition-gazebo-imu-system" name="ignition::gazebo::systems::Imu">
+      </plugin>
+      <plugin filename="ignition-gazebo-sensors-system" name="ignition::gazebo::systems::Sensors">
+        <render_engine>ogre2</render_engine>
+      </plugin>
+    </xacro:if>
+    <!-- ROS 2 Iron or above -->
+    <xacro:unless value="$(arg is_ignition)">
+      <plugin filename="gz_ros2_control-system" name="gz_ros2_control::GazeboSimROS2ControlPlugin">
+        <parameters>$(find bumperbot_controller)/config/bumperbot_controllers.yaml</parameters>
+      </plugin>
+      <plugin filename="gz-sim-imu-system" name="gz::sim::systems::Imu">
+      </plugin>
+      <plugin filename="gz-sim-sensors-system" name="gz::sim::systems::Sensors">
+        <render_engine>ogre2</render_engine>
+      </plugin>
+    </xacro:unless>
   </gazebo>
   <!-- IMU -->
@@ -75,4 +67,6 @@
         <always_on>true</always_on>
         <update_rate>100</update_rate>
+        <gz_frame_id>imu_link</gz_frame_id>
+        <topic>imu</topic>
         <imu>
           <angular_velocity>
@@ -117,14 +111,15 @@
           </linear_acceleration>
         </imu>
-        <plugin name="imu" filename="libgazebo_ros_imu_sensor.so"/>
     </sensor>
   </gazebo>
   <!-- 2D Laser Sensor -->
   <gazebo reference="laser_link">
-    <sensor name="lidar" type="ray">
+    <sensor name="lidar" type="gpu_lidar">
       <always_on>true</always_on>
       <visualize>true</visualize>
+      <topic>scan</topic>
       <update_rate>5</update_rate>
-      <ray>
+      <gz_frame_id>laser_link</gz_frame_id>
+      <lidar>
         <scan>
           <horizontal>
@@ -145,12 +140,5 @@
           <stddev>0.01</stddev>
         </noise>
-      </ray>
-      <plugin name="scan" filename="libgazebo_ros_ray_sensor.so">
-        <ros>
-          <remapping>~/out:=scan</remapping>
-        </ros>
-        <output_type>sensor_msgs/LaserScan</output_type>
-        <frame_name>laser_link</frame_name>
-      </plugin>
+      </lidar>
     </sensor>
   </gazebo>

File: Section9_Localization_with_known_Map/bumperbot_ws/src/bumperbot_description/urdf/bumperbot_ros2_control.xacro (robot description, xacro)
@@ -4,7 +4,16 @@
         <!-- ros2_control Gazebo -->
         <xacro:if value="$(arg is_sim)">
-            <hardware>
-                <plugin>gazebo_ros2_control/GazeboSystem</plugin>
-            </hardware>
+            <!-- ROS 2 Humble -->
+            <xacro:if value="$(arg is_ignition)">
+                <hardware>
+                    <plugin>ign_ros2_control/IgnitionSystem</plugin>
+                </hardware>
+            </xacro:if>
+            <!-- ROS 2 Iron or above -->
+            <xacro:unless value="$(arg is_ignition)">
+                <hardware>
+                    <plugin>gz_ros2_control/GazeboSimSystem</plugin>
+                </hardware>
+            </xacro:unless>
         </xacro:if>
         <!-- ros2_control Real Robot -->
